Commit message: some additional updates

File: src/ros2_bot_description/urdf/ros2bot.urdf.xacro (robot description, xacro)
@@ -7,8 +7,16 @@
     <xacro:property name="scale" value="0.01 0.01 0.01"/>
     <!--rpy stand for Radians Pitch and Yaw xyz = axis directions  -->
+    <!-- creating a macro function so I dont have to repeate code using xacro:macro -->
+     <xacro:macro name="default_inertial" params="mass">
+        <intertial>
+            <mass value ="${mass}" /><!--passing in param of mass-->
+            <inertia ixx="0.0" ixy="0.0" ixz="0.0" iyy="1.0" iyz="0.0" izz="1.0"/>
+        </intertial>
+     </xacro:macro>
     <!-- Define world link -->
     <link name="world"/>
     <!-- Define base link -->
     <link name="base_link">
+        <xacro:default_inert mass="1.0"/>
         <visual>
             <origin rpy="0 0 0" xyz="-0.5 -0.5 0"/>
@@ -17,4 +25,10 @@
             </geometry>
         </visual>
+        <collision>
+            <origin rpy="0 0 0" xyz="-0.5 -0.5 0"/>
+            <geometry>
+                <mesh filename="package://ros2_bot_description/meshes/basement.STL" scale="${scale}"/>
+            </geometry>
+        </collision>
     </link>
     <!-- Define virtual joint -->
@@ -26,4 +40,5 @@
     <!-- Define base plate link -->
     <link name="base_plate">
+        <xacro:default_inert mass="0.1"/>
         <visual>
             <origin rpy="0 0 0" xyz="-0.39 -0.39 -0.56"/>
@@ -32,4 +47,10 @@
             </geometry>
         </visual>
+        <collision>
+            <origin rpy="0 0 0" xyz="-0.39 -0.39 -0.56"/>
+            <geometry>
+                <mesh filename="package://ros2_bot_description/meshes/base_plate.STL" scale="${scale}"/>
+            </geometry>
+        </collision>
     </link>
     <!-- Define joint1 -->
@@ -43,4 +64,5 @@
     <!-- Define forward drive arm link -->
     <link name="forward_drive_arm">
+        <xacro:default_inert mass="0.1"/>
         <visual>
             <origin rpy="0 -${PI / 2} ${PI / 2}" xyz="0.19 0.06 -0.08"/>
@@ -49,4 +71,10 @@
             </geometry>
         </visual>
+        <collision>
+            <origin rpy="0 -${PI / 2} ${PI / 2}" xyz="0.19 0.06 -0.08"/>
+            <geometry>
+                <mesh filename="package://ros2_bot_description/meshes/forward_drive_arm.STL" scale="${scale}"/>
+            </geometry>
+        </collision>
     </link>
     <!-- Define joint2 -->
@@ -61,4 +89,5 @@
     <link name="horizontal_arm">
         <visual>
+            <xacro:default_inert mass="0.1"/>
             <origin rpy="-${PI / 2} 0 ${PI / 2}" xyz="-0.03 -0.4 -0.06"/>
             <geometry>
@@ -66,4 +95,10 @@
             </geometry>
         </visual>
+        <collision>
+            <origin rpy="-${PI / 2} 0 ${PI / 2}" xyz="-0.03 -0.4 -0.06"/>
+            <geometry>
+                <mesh filename="package://ros2_bot_description/meshes/horizontal_arm.STL" scale="${scale}"/>
+            </geometry>
+        </collision>
     </link>
     <!-- Define joint3 -->
@@ -77,4 +112,5 @@
     <!-- Define claw support link -->
     <link name="claw_support">
+        <xacro:default_inert mass="0.05"/>
         <visual>
             <origin rpy="0 0 ${PI / 2}" xyz="0 -0.05 -0.15"/>
@@ -83,4 +119,10 @@
             </geometry>
         </visual>
+        <collision>
+            <origin rpy="0 0 ${PI / 2}" xyz="0 -0.05 -0.15"/>
+            <geometry>
+                <mesh filename="package://ros2_bot_description/meshes/claw_support.STL" scale="${scale}"/>
+            </geometry>
+        </collision>
     </link>
     <!-- Define joint4 -->
@@ -92,4 +134,5 @@
     <!-- Define right finger link -->
     <link name="right_finger">
+        <xacro:default_inert mass="0.01"/>
         <visual>
             <origin rpy="0 0 -${PI / 2}" xyz="-0.1 0.5 -0.1"/>
@@ -98,4 +141,10 @@
             </geometry>
         </visual>
+        <collision>
+            <origin rpy="0 0 -${PI / 2}" xyz="-0.1 0.5 -0.1"/>
+            <geometry>
+                <mesh filename="package://ros2_bot_description/meshes/right_finger.STL" scale="${scale}"/>
+            </geometry>
+        </collision>
     </link>
     <!-- Define joint5 -->
@@ -109,4 +158,5 @@
     <!-- Define left finger link -->
     <link name="left_finger">
+        <xacro:default_inert mass="0.01"/>
         <visual>
             <origin rpy="0 0 -${PI / 2}" xyz="-0.04 0.5 -0.1"/>
@@ -115,4 +165,10 @@
             </geometry>
         </visual>
+        <collision>
+            <origin rpy="0 0 -${PI / 2}" xyz="-0.04 0.5 -0.1"/>
+            <geometry>
+                <mesh filename="package://ros2_bot_description/meshes/left_finger.STL" scale="${scale}"/>
+            </geometry>
+        </collision>
     </link>
     <!-- Define joint6 -->
@@ -125,6 +181,7 @@
         <mimic joint="joint5" multiplier="-1"/>
     </joint>
-    Camera plate
+    <!-- Camera plate -->
     <link name="rgb_camera">
+        <xacro:default_inert mass="0.1"/>
         <visual>
             <origin rpy="0.2 -0.06 -1.6" xyz="-0.12 0.12 -0.1"/> <!-- Adjusted values -->
@@ -133,4 +190,10 @@
             </geometry>
         </visual>
+        <collision>
+            <origin rpy="0.2 -0.06 -1.6" xyz="-0.12 0.12 -0.1"/> <!-- Adjusted values -->
+            <geometry>
+                <mesh filename="package://ros2_bot_description/meshes/pi_camera.STL" scale="${scale}"/>
+            </geometry>
+        </collision>
     </link>
     <joint name="rgb_camera_joint" type="fixed">
