Commit message: working bot full out line

File: install/ros2_bot_description/share/ros2_bot_description/urdf/ros2bot.urdf.xacro (robot description, xacro)
@@ -1,16 +1,21 @@
 <?xml version="1.0"?>
 <robot xmlns:xacro="http://www.ros.org/wiki/xacro" name="ros2bot">
+    <!-- Define properties for reuse -->
     <xacro:property name="PI" value="3.14159"/>
     <xacro:property name="effort" value="30.0"/>
     <xacro:property name="velocity" value="10.0"/>
+    <xacro:property name="scale" value="0.01 0.01 0.01"/>
+    <!-- Define world link -->
     <link name="world"/>
+    <!-- Define base link -->
     <link name="base_link">
         <visual>
             <origin rpy="0 0 0" xyz="-0.5 -0.5 0"/>
             <geometry>
-                <mesh filename="package://ros2_bot_description/meshes/basement.STL" scale="0.01 0.01 0.01"/>
+                <mesh filename="package://ros2_bot_description/meshes/basement.STL" scale="${scale}"/>
             </geometry>
         </visual>
     </link>
+    <!-- Define virtual joint -->
     <joint name="virtual_joint" type="fixed">
         <parent link="world"/>
@@ -18,18 +23,104 @@
         <origin rpy="0 0 0" xyz="0 0 0"/>
     </joint>
+    <!-- Define base plate link -->
     <link name="base_plate">
         <visual>
             <origin rpy="0 0 0" xyz="-0.39 -0.39 -0.56"/>
             <geometry>
-                <mesh filename="package://ros2_bot_description/meshes/base_plate.STL" scale="0.01 0.01 0.01"/>
+                <mesh filename="package://ros2_bot_description/meshes/base_plate.STL" scale="${scale}"/>
             </geometry>
         </visual>
     </link>
+    <!-- Define joint1 -->
     <joint name="joint1" type="revolute">
         <parent link="base_link"/>
         <child link="base_plate"/>
-        <axis xyz="0 0 1" />
+        <axis xyz="0 0 1"/>
         <origin rpy="0 0 0" xyz="0 0 0.307"/>
-        <limit lower="-${PI/2}" upper="${PI/2}" effort="${effort}"  velocity="${velocity}"/>
+        <limit lower="-${PI/2}" upper="${PI/2}" effort="${effort}" velocity="${velocity}"/>
+    </joint>
+    <!-- Define forward drive arm link -->
+    <link name="forward_drive_arm">
+        <visual>
+            <origin rpy="0 -${PI / 2} ${PI / 2}" xyz="0.19 0.06 -0.08"/>
+            <geometry>
+                <mesh filename="package://ros2_bot_description/meshes/forward_drive_arm.STL" scale="${scale}"/>
+            </geometry>
+        </visual>
+    </link>
+    <!-- Define joint2 -->
+    <joint name="joint2" type="revolute">
+        <parent link="base_plate"/>
+        <child link="forward_drive_arm"/>
+        <axis xyz="1 0 0"/>
+        <origin rpy="0 0 0" xyz="-0.02 0 0.35"/>
+        <limit lower="-${PI/2}" upper="${PI/2}" effort="${effort}" velocity="${velocity}"/>
+    </joint>
+    <!-- Define horizontal arm link -->
+    <link name="horizontal_arm">
+        <visual>
+            <origin rpy="-${PI / 2} 0 ${PI / 2}" xyz="-0.03 -0.4 -0.06"/>
+            <geometry>
+                <mesh filename="package://ros2_bot_description/meshes/horizontal_arm.STL" scale="${scale}"/>
+            </geometry>
+        </visual>
+    </link>
+    <!-- Define joint3 -->
+    <joint name="joint3" type="revolute">
+        <parent link="forward_drive_arm"/>
+        <child link="horizontal_arm"/>
+        <axis xyz="1 0 0"/>
+        <origin rpy="0 0 0" xyz="0 0 0.8"/>
+        <limit lower="-${PI/2}" upper="${PI/2}" effort="${effort}" velocity="${velocity}"/>
+    </joint>
+    <!-- Define claw support link -->
+    <link name="claw_support">
+        <visual>
+            <origin rpy="0 0 ${PI / 2}" xyz="0 -0.05 -0.15"/>
+            <geometry>
+                <mesh filename="package://ros2_bot_description/meshes/claw_support.STL" scale="${scale}"/>
+            </geometry>
+        </visual>
+    </link>
+    <!-- Define joint4 -->
+    <joint name="joint4" type="fixed">
+        <parent link="horizontal_arm"/>
+        <child link="claw_support"/>
+        <origin rpy="0 0 0" xyz="0 0.82 0"/>
+    </joint>
+    <!-- Define right finger link -->
+    <link name="right_finger">
+        <visual>
+            <origin rpy="0 0 -${PI / 2}" xyz="-0.1 0.5 -0.1"/>
+            <geometry>
+                <mesh filename="package://ros2_bot_description/meshes/right_finger.STL" scale="${scale}"/>
+            </geometry>
+        </visual>
+    </link>
+    <!-- Define joint5 -->
+    <joint name="joint5" type="revolute">
+        <parent link="claw_support"/>
+        <child link="right_finger"/>
+        <axis xyz="0 0 1"/>
+        <origin rpy="0 0 0" xyz="-0.04 0.13 -0.1"/>
+        <limit lower="-${PI/2}" upper="0.0" effort="${effort}" velocity="${velocity}"/>
+    </joint>
+    <!-- Define left finger link -->
+    <link name="left_finger">
+        <visual>
+            <origin rpy="0 0 -${PI / 2}" xyz="-0.04 0.5 -0.1"/>
+            <geometry>
+                <mesh filename="package://ros2_bot_description/meshes/left_finger.STL" scale="${scale}"/>
+            </geometry>
+        </visual>
+    </link>
+    <!-- Define joint6 -->
+    <joint name="joint6" type="revolute">
+        <parent link="claw_support"/>
+        <child link="left_finger"/>
+        <axis xyz="0 0 1"/>
+        <origin rpy="0 0 0" xyz="-0.22 0.13 -0.1"/>
+        <limit lower="0.0" upper="${PI/2}" effort="${effort}" velocity="${velocity}"/>
+        <mimic joint="joint5" multiplier="-1"/>
     </joint>
 </robot>

Commit message: changes made

File: install/ros2_bot_description/share/ros2_bot_description/urdf/ros2bot.urdf.xacro (robot description, xacro)
@@ -6,4 +6,5 @@
     <xacro:property name="velocity" value="10.0"/>
     <xacro:property name="scale" value="0.01 0.01 0.01"/>
+    <!--rpy stand for Radians Pitch and Yaw xyz = axis directions  -->
     <!-- Define world link -->
     <link name="world"/>
@@ -124,3 +125,17 @@
         <mimic joint="joint5" multiplier="-1"/>
     </joint>
+    Camera plate
+    <link name="rgb_camera">
+        <visual>
+            <origin rpy="-${PI/2.0} 0 -${PI/2.0}" xyz="-0.12 0.12 -0.1"/> <!-- Adjusted values -->
+            <geometry>
+                <mesh filename="package://ros2_bot_description/meshes/pi_camera.STL" scale="${scale}"/>
+            </geometry>
+        </visual>
+    </link>
+    <joint name="rgb_camera_joint" type="fixed">
+        <parent link="base_link"/>
+        <child link="rgb_camera"/>
+        <origin rpy="0 1.5 1.4" xyz="0 0.43 0.18"/>
+    </joint>
 </robot>

File: src/ros2_bot_description/urdf/ros2bot.urdf.xacro (robot description, xacro)
@@ -6,4 +6,5 @@
     <xacro:property name="velocity" value="10.0"/>
     <xacro:property name="scale" value="0.01 0.01 0.01"/>
+    <!--rpy stand for Radians Pitch and Yaw xyz = axis directions  -->
     <!-- Define world link -->
     <link name="world"/>
@@ -124,3 +125,17 @@
         <mimic joint="joint5" multiplier="-1"/>
     </joint>
+    Camera plate
+    <link name="rgb_camera">
+        <visual>
+            <origin rpy="0.2 -0.06 -1.6" xyz="-0.12 0.12 -0.1"/> <!-- Adjusted values -->
+            <geometry>
+                <mesh filename="package://ros2_bot_description/meshes/pi_camera.STL" scale="${scale}"/>
+            </geometry>
+        </visual>
+    </link>
+    <joint name="rgb_camera_joint" type="fixed">
+        <parent link="base_link"/>
+        <child link="rgb_camera"/>
+        <origin rpy="0 1.5 1.4" xyz="0 0.43 0.18"/>
+    </joint>
 </robot>

Commit message: updated files

File: install/ros2_bot_description/share/ros2_bot_description/urdf/ros2bot.urdf.xacro (robot description, xacro)
@@ -7,8 +7,17 @@
     <xacro:property name="scale" value="0.01 0.01 0.01"/>
     <!--rpy stand for Radians Pitch and Yaw xyz = axis directions  -->
+    <!-- creating a macro function so I dont have to repeate code using xacro:macro -->
+    <xacro:macro name="default_inertial" params="mass">
+        <inertial>
+          <mass value="${mass}" />
+          <inertia ixx="1.0" ixy="0.0" ixz="0.0"
+                    iyy="1.0" iyz="0.0" izz="1.0" />
+        </inertial>
+    </xacro:macro>
     <!-- Define world link -->
     <link name="world"/>
     <!-- Define base link -->
     <link name="base_link">
+        <xacro:default_inertial mass="1.0"/>
         <visual>
             <origin rpy="0 0 0" xyz="-0.5 -0.5 0"/>
@@ -17,4 +26,10 @@
             </geometry>
         </visual>
+        <collision>
+            <origin rpy="0 0 0" xyz="-0.5 -0.5 0"/>
+            <geometry>
+                <mesh filename="package://ros2_bot_description/meshes/basement.STL" scale="${scale}"/>
+            </geometry>
+        </collision>
     </link>
     <!-- Define virtual joint -->
@@ -26,4 +41,5 @@
     <!-- Define base plate link -->
     <link name="base_plate">
+        <xacro:default_inertial mass="0.1"/>
         <visual>
             <origin rpy="0 0 0" xyz="-0.39 -0.39 -0.56"/>
@@ -32,4 +48,10 @@
             </geometry>
         </visual>
+        <collision>
+            <origin rpy="0 0 0" xyz="-0.39 -0.39 -0.56"/>
+            <geometry>
+                <mesh filename="package://ros2_bot_description/meshes/base_plate.STL" scale="${scale}"/>
+            </geometry>
+        </collision>
     </link>
     <!-- Define joint1 -->
@@ -43,4 +65,5 @@
     <!-- Define forward drive arm link -->
     <link name="forward_drive_arm">
+        <xacro:default_inertial mass="0.1"/>
         <visual>
             <origin rpy="0 -${PI / 2} ${PI / 2}" xyz="0.19 0.06 -0.08"/>
@@ -49,4 +72,10 @@
             </geometry>
         </visual>
+        <collision>
+            <origin rpy="0 -${PI / 2} ${PI / 2}" xyz="0.19 0.06 -0.08"/>
+            <geometry>
+                <mesh filename="package://ros2_bot_description/meshes/forward_drive_arm.STL" scale="${scale}"/>
+            </geometry>
+        </collision>
     </link>
     <!-- Define joint2 -->
@@ -61,4 +90,5 @@
     <link name="horizontal_arm">
         <visual>
+            <xacro:default_inertial mass="0.1"/>
             <origin rpy="-${PI / 2} 0 ${PI / 2}" xyz="-0.03 -0.4 -0.06"/>
             <geometry>
@@ -66,4 +96,10 @@
             </geometry>
         </visual>
+        <collision>
+            <origin rpy="-${PI / 2} 0 ${PI / 2}" xyz="-0.03 -0.4 -0.06"/>
+            <geometry>
+                <mesh filename="package://ros2_bot_description/meshes/horizontal_arm.STL" scale="${scale}"/>
+            </geometry>
+        </collision>
     </link>
     <!-- Define joint3 -->
@@ -77,4 +113,5 @@
     <!-- Define claw support link -->
     <link name="claw_support">
+        <xacro:default_inertial mass="0.05"/>
         <visual>
             <origin rpy="0 0 ${PI / 2}" xyz="0 -0.05 -0.15"/>
@@ -83,4 +120,10 @@
             </geometry>
         </visual>
+        <collision>
+            <origin rpy="0 0 ${PI / 2}" xyz="0 -0.05 -0.15"/>
+            <geometry>
+                <mesh filename="package://ros2_bot_description/meshes/claw_support.STL" scale="${scale}"/>
+            </geometry>
+        </collision>
     </link>
     <!-- Define joint4 -->
@@ -89,7 +132,8 @@
         <child link="claw_support"/>
         <origin rpy="0 0 0" xyz="0 0.82 0"/>
-    </joint>
+    </joint>﻿⁠server-roles﻿
     <!-- Define right finger link -->
     <link name="right_finger">
+        <xacro:default_inertial mass="0.01"/>
         <visual>
             <origin rpy="0 0 -${PI / 2}" xyz="-0.1 0.5 -0.1"/>
@@ -98,4 +142,10 @@
             </geometry>
         </visual>
+        <collision>
+            <origin rpy="0 0 -${PI / 2}" xyz="-0.1 0.5 -0.1"/>
+            <geometry>
+                <mesh filename="package://ros2_bot_description/meshes/right_finger.STL" scale="${scale}"/>
+            </geometry>
+        </collision>
     </link>
     <!-- Define joint5 -->
@@ -109,4 +159,5 @@
     <!-- Define left finger link -->
     <link name="left_finger">
+        <xacro:default_inertial mass="0.01"/>
         <visual>
             <origin rpy="0 0 -${PI / 2}" xyz="-0.04 0.5 -0.1"/>
@@ -115,4 +166,10 @@
             </geometry>
         </visual>
+        <collision>
+            <origin rpy="0 0 -${PI / 2}" xyz="-0.04 0.5 -0.1"/>
+            <geometry>
+                <mesh filename="package://ros2_bot_description/meshes/left_finger.STL" scale="${scale}"/>
+            </geometry>
+        </collision>
     </link>
     <!-- Define joint6 -->
@@ -125,12 +182,22 @@
         <mimic joint="joint5" multiplier="-1"/>
     </joint>
-    Camera plate
+    <!-- Camera plate -->
     <link name="rgb_camera">
-        <visual>
-            <origin rpy="-${PI/2.0} 0 -${PI/2.0}" xyz="-0.12 0.12 -0.1"/> <!-- Adjusted values -->
+        <xacro:default_inertial mass="0.1"/>
+        <visual>
+            <origin rpy="0.2 -0.06 -1.6" xyz="-0.12 0.12 -0.1"/> <!-- Adjusted values -->
             <geometry>
                 <mesh filename="package://ros2_bot_description/meshes/pi_camera.STL" scale="${scale}"/>
             </geometry>
         </visual>
+        <collision>
+            <gazebo>
+                <sensor type="camera" name="rgb_camera_sensor">
+                    <always_on>0</always_on>
+                    <update_rate>1</update_rate>
+                    <camera name="rgb_camera"/>
+                </sensor>
+            </gazebo>
+        </collision>
     </link>
     <joint name="rgb_camera_joint" type="fixed">

File: src/ros2_bot_description/urdf/ros2bot.urdf.xacro (robot description, xacro)
@@ -8,15 +8,16 @@
     <!--rpy stand for Radians Pitch and Yaw xyz = axis directions  -->
     <!-- creating a macro function so I dont have to repeate code using xacro:macro -->
-     <xacro:macro name="default_inertial" params="mass">
-        <intertial>
-            <mass value ="${mass}" /><!--passing in param of mass-->
-            <inertia ixx="0.0" ixy="0.0" ixz="0.0" iyy="1.0" iyz="0.0" izz="1.0"/>
-        </intertial>
-     </xacro:macro>
+    <xacro:macro name="default_inertial" params="mass">
+        <inertial>
+          <mass value="${mass}" />
+          <inertia ixx="1.0" ixy="0.0" ixz="0.0"
+                    iyy="1.0" iyz="0.0" izz="1.0" />
+        </inertial>
+    </xacro:macro>
     <!-- Define world link -->
     <link name="world"/>
     <!-- Define base link -->
     <link name="base_link">
-        <xacro:default_inert mass="1.0"/>
+        <xacro:default_inertial mass="1.0"/>
         <visual>
             <origin rpy="0 0 0" xyz="-0.5 -0.5 0"/>
@@ -40,5 +41,5 @@
     <!-- Define base plate link -->
     <link name="base_plate">
-        <xacro:default_inert mass="0.1"/>
+        <xacro:default_inertial mass="0.1"/>
         <visual>
             <origin rpy="0 0 0" xyz="-0.39 -0.39 -0.56"/>
@@ -64,5 +65,5 @@
     <!-- Define forward drive arm link -->
     <link name="forward_drive_arm">
-        <xacro:default_inert mass="0.1"/>
+        <xacro:default_inertial mass="0.1"/>
         <visual>
             <origin rpy="0 -${PI / 2} ${PI / 2}" xyz="0.19 0.06 -0.08"/>
@@ -89,5 +90,5 @@
     <link name="horizontal_arm">
         <visual>
-            <xacro:default_inert mass="0.1"/>
+            <xacro:default_inertial mass="0.1"/>
             <origin rpy="-${PI / 2} 0 ${PI / 2}" xyz="-0.03 -0.4 -0.06"/>
             <geometry>
@@ -112,5 +113,5 @@
     <!-- Define claw support link -->
     <link name="claw_support">
-        <xacro:default_inert mass="0.05"/>
+        <xacro:default_inertial mass="0.05"/>
         <visual>
             <origin rpy="0 0 ${PI / 2}" xyz="0 -0.05 -0.15"/>
@@ -131,8 +132,8 @@
         <child link="claw_support"/>
         <origin rpy="0 0 0" xyz="0 0.82 0"/>
-    </joint>
+    </joint>﻿⁠server-roles﻿
     <!-- Define right finger link -->
     <link name="right_finger">
-        <xacro:default_inert mass="0.01"/>
+        <xacro:default_inertial mass="0.01"/>
         <visual>
             <origin rpy="0 0 -${PI / 2}" xyz="-0.1 0.5 -0.1"/>
@@ -158,5 +159,5 @@
     <!-- Define left finger link -->
     <link name="left_finger">
-        <xacro:default_inert mass="0.01"/>
+        <xacro:default_inertial mass="0.01"/>
         <visual>
             <origin rpy="0 0 -${PI / 2}" xyz="-0.04 0.5 -0.1"/>
@@ -183,5 +184,5 @@
     <!-- Camera plate -->
     <link name="rgb_camera">
-        <xacro:default_inert mass="0.1"/>
+        <xacro:default_inertial mass="0.1"/>
         <visual>
             <origin rpy="0.2 -0.06 -1.6" xyz="-0.12 0.12 -0.1"/> <!-- Adjusted values -->
@@ -191,8 +192,11 @@
         </visual>
         <collision>
-            <origin rpy="0.2 -0.06 -1.6" xyz="-0.12 0.12 -0.1"/> <!-- Adjusted values -->
-            <geometry>
-                <mesh filename="package://ros2_bot_description/meshes/pi_camera.STL" scale="${scale}"/>
-            </geometry>
+            <gazebo>
+                <sensor type="camera" name="rgb_camera_sensor">
+                    <always_on>0</always_on>
+                    <update_rate>1</update_rate>
+                    <camera name="rgb_camera"/>
+                </sensor>
+            </gazebo>
         </collision>
     </link>
